File: HW/USB_Telegraph.kicad_sch (KiCad schematic)
At the start: 34 parts, among them J1 USB_C_Receptacle_USB2.0, J2 Conn_02x05_Odd_Even, J3 Screw_Terminal_01x01, J4 Screw_Terminal_01x01, J5 Conn_01x03, Q1 NP2302FVR, U1 STM32F103C8Tx, U2 XC6206PxxxMR, U4 USBLC6-2SC6, Y1 8MHz

Commit message: Initial routing
Parts:
- J1: footprint Connector_USB:USB_C_Receptacle_G-Switch_GT-USB-7010ASV -> Connectors:USB_C_Receptacle_G-Switch_GT-USB-7010ASV
- RV1: PN VG039NCHXTB102 -> VG039NCHXTB101
Connections:
- net GND: now also J1.S1 (SHIELD), J5.3 (Pin_3)
- net SWDCLK: now also J5.2 (Pin_2)
- net SWDIO: now also J5.1 (Pin_1)
- net USB_DM renamed USB_DN
- net USB_DM_ST renamed USB_ST_DN
- net USB_DP_ST renamed USB_ST_DP
Other:
- moved on the sheet: J5
Changed lines of the file:
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@@
   (junction (at 132.08 45.72) (diameter 0) (color 0 0 0 0)
   )
+  (junction (at 35.56 111.76) (diameter 0) (color 0 0 0 0)
+  )
   (junction (at 67.31 81.28) (diameter 0) (color 0 0 0 0)
   )
@@
     (stroke (width 0) (type default))
   )
+  (wire (pts (xy 46.99 132.08) (xy 39.37 132.08))
+    (stroke (width 0) (type default))
+  )
   (wire (pts (xy 53.34 91.44) (xy 53.34 93.98))
     (stroke (width 0) (type default))
@@
     (stroke (width 0) (type default))
   )
+  (wire (pts (xy 39.37 134.62) (xy 46.99 134.62))
+    (stroke (width 0) (type default))
+  )
   (wire (pts (xy 120.65 53.34) (xy 120.65 54.61))
     (stroke (width 0) (type default))
@@
     (stroke (width 0) (type default))
   )
+  (wire (pts (xy 27.94 111.76) (xy 35.56 111.76))
+    (stroke (width 0) (type default))
+  )
   (wire (pts (xy 67.31 81.28) (xy 67.31 82.55))
     (stroke (width 0) (type default))
@@
     (stroke (width 0) (type default))
   )
-  (label "USB_DP_ST" (at 100.33 101.6 0) (fields_autoplaced)
+  (label "USB_ST_DP" (at 100.33 101.6 0) (fields_autoplaced)
     (effects (font (size 1.27 1.27)) (justify left bottom))
   )
-  (label "USB_DM" (at 80.01 96.52 180) (fields_autoplaced)
+  (label "USB_DN" (at 80.01 96.52 180) (fields_autoplaced)
     (effects (font (size 1.27 1.27)) (justify right bottom))
   )
@@
     (effects (font (size 1.27 1.27)) (justify left bottom))
   )
-  (label "USB_DM" (at 63.5 88.9 180) (fields_autoplaced)
+  (label "USB_DN" (at 63.5 88.9 180) (fields_autoplaced)
     (effects (font (size 1.27 1.27)) (justify right bottom))
   )
-  (label "USB_DM_ST" (at 80.01 101.6 180) (fields_autoplaced)
+  (label "USB_ST_DN" (at 80.01 101.6 180) (fields_autoplaced)
     (effects (font (size 1.27 1.27)) (justify right bottom))
+  )
+  (label "SWDIO" (at 39.37 132.08 0) (fields_autoplaced)
+    (effects (font (size 1.27 1.27)) (justify left bottom))
   )
   (label "SWO" (at 66.04 161.29 180) (fields_autoplaced)
@@
     (effects (font (size 1.27 1.27)) (justify left bottom))
   )
+  (label "SWDCLK" (at 39.37 134.62 0) (fields_autoplaced)
+    (effects (font (size 1.27 1.27)) (justify left bottom))
+  )
   (label "SENSE2" (at 217.17 88.9 0) (fields_autoplaced)
     (effects (font (size 1.27 1.27)) (justify left bottom))
   )
-  (label "USB_DM_ST" (at 198.12 73.66 180) (fields_autoplaced)
+  (label "USB_ST_DN" (at 198.12 73.66 180) (fields_autoplaced)
     (effects (font (size 1.27 1.27)) (justify right bottom))
   )
@@
     (effects (font (size 1.27 1.27)) (justify left bottom))
   )
-  (label "USB_DP_ST" (at 198.12 76.2 180) (fields_autoplaced)
+  (label "USB_ST_DP" (at 198.12 76.2 180) (fields_autoplaced)
     (effects (font (size 1.27 1.27)) (justify right bottom))
   )
@@
       (effects (font (size 1.27 1.27)) hide)
     )
-    (property "PN" "VG039NCHXTB102" (at 248.92 93.98 0)
+    (property "PN" "VG039NCHXTB101" (at 248.92 93.98 0)
       (effects (font (size 1.27 1.27)) hide)
     )
@@
     )
   )
+  (symbol (lib_id "power:GND") (at 46.99 137.16 0) (unit 1)
+    (in_bom yes) (on_board yes) (dnp no)
+    (property "Reference" "#PWR028" (at 46.99 143.51 0)
+      (effects (font (size 1.27 1.27)) hide)
+    )
+    (property "Value" "GND" (at 43.18 138.43 0)
+      (effects (font (size 1.27 1.27)))
+    )
+    (property "Footprint" "" (at 46.99 137.16 0)
+      (effects (font (size 1.27 1.27)) hide)
+    )
+    (property "Datasheet" "" (at 46.99 137.16 0)
+      (effects (font (size 1.27 1.27)) hide)
+    )
+    (pin "1")
+    (instances
+      (project "USB_Telegraph"
+        (path "/7a47d1a4-76a9-416d-b989-2852c78f231c"
+          (reference "#PWR028") (unit 1)
+        )
+      )
+    )
+  )
   (symbol (lib_id "power:+3V3") (at 39.37 151.13 0) (unit 1)
     (in_bom yes) (on_board yes) (dnp no) (fields_autoplaced)
@@
       (effects (font (size 1.27 1.27)))
     )
-    (property "Footprint" "Connector_USB:USB_C_Receptacle_G-Switch_GT-USB-7010ASV" (at 39.37 88.9 0)
+    (property "Footprint" "Connectors:USB_C_Receptacle_G-Switch_GT-USB-7010ASV" (at 39.37 88.9 0)
       (effects (font (size 1.27 1.27)) hide)
     )
@@
     )
   )
-  (symbol (lib_id "Connector_Generic:Conn_01x03") (at 52.07 139.7 0) (unit 1)
-    (in_bom yes) (on_board yes) (dnp no) (fields_autoplaced)
-    (property "Reference" "J5" (at 54.61 138.43 0)
-      (effects (font (size 1.27 1.27)) (justify left))
-    )
-    (property "Value" "Conn_01x03" (at 54.61 140.97 0)
-      (effects (font (size 1.27 1.27)) (justify left))
-    )
-    (property "Footprint" "Connector_PinSocket_2.54mm:PinSocket_1x03_P2.54mm_Horizontal" (at 52.07 139.7 0)
-      (effects (font (size 1.27 1.27)) hide)
-    )
-    (property "Datasheet" "~" (at 52.07 139.7 0)
-      (effects (font (size 1.27 1.27)) hide)
-    )
+  (symbol (lib_id "Connector_Generic:Conn_01x03") (at 52.07 134.62 0) (unit 1)
+    (in_bom yes) (on_board yes) (dnp no) (fields_autoplaced)
+    (property "Reference" "J5" (at 54.61 133.35 0)
+      (effects (font (size 1.27 1.27)) (justify left))
+    )
+    (property "Value" "Conn_01x03" (at 54.61 135.89 0)
+      (effects (font (size 1.27 1.27)) (justify left))
+    )
+    (property "Footprint" "Connector_PinSocket_2.54mm:PinSocket_1x03_P2.54mm_Horizontal" (at 52.07 134.62 0)
+      (effects (font (size 1.27 1.27)) hide)
+    )
+    (property "Datasheet" "~" (at 52.07 134.62 0)
+      (effects (font (size 1.27 1.27)) hide)
+    )

Commit message: Routing done, part assignement done
Parts:
- C1, C2: PN (none) -> CC0402JRNPO9BN220
- C10, C3, C4, C5, C6: PN (none) -> CC0402KRX7R7BB104
- C7: PN (none) -> CC0402KRX5R6BB475
- C8: PN (none) -> CC0402ZRY5V6BB105
- J5: PN (none) -> DNP
- R1, R12, R13, R8, R9: PN (none) -> RC0402FR-0710KL
- R11, R7: PN (none) -> RC0402FR-071K5L
- R2: PN (none) -> RC0402FR-071ML
- R3, R4: PN (none) -> RC0402FR-0722RL
- R5, R6: PN (none) -> RC0402FR-075K1L
- RV1: footprint Potentiometer_SMD:Potentiometer_Bourns_TC33X_Vertical -> Potentiometer_SMD:Potentiometer_Bourns_3314J_Vertical; PN VG039NCHXTB101 -> 3314J-1-101E
Changed lines of the file:
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@@
+      (effects (font (size 1.27 1.27)) hide)
+    )
+    (property "PN" "RC0402FR-071K5L" (at 233.68 106.68 0)
       (effects (font (size 1.27 1.27)) hide)
     )
@@
       (effects (font (size 1.27 1.27)) hide)
     )
+    (property "PN" "RC0402FR-0710KL" (at 232.41 71.12 0)
+      (effects (font (size 1.27 1.27)) hide)
+    )
     (pin "1")
     (pin "2")
@@
       (effects (font (size 1.27 1.27)) hide)
     )
+    (property "PN" "RC0402FR-075K1L" (at 58.42 78.74 0)
+      (effects (font (size 1.27 1.27)) hide)
+    )
     (pin "1")
     (pin "2")
@@
       (effects (font (size 1.27 1.27)) (justify right))
     )
-    (property "Footprint" "Potentiometer_SMD:Potentiometer_Bourns_TC33X_Vertical" (at 248.92 93.98 0)
+    (property "Footprint" "Potentiometer_SMD:Potentiometer_Bourns_3314J_Vertical" (at 248.92 93.98 0)
       (effects (font (size 1.27 1.27)) hide)
     )
@@
       (effects (font (size 1.27 1.27)) hide)
     )
-    (property "PN" "VG039NCHXTB101" (at 248.92 93.98 0)
+    (property "PN" "3314J-1-101E" (at 248.92 93.98 0)
       (effects (font (size 1.27 1.27)) hide)
     )
@@
       (effects (font (size 1.27 1.27)) hide)
     )
+    (property "PN" "RC0402FR-0710KL" (at 232.41 92.71 0)
+      (effects (font (size 1.27 1.27)) hide)
+    )
     (pin "1")
     (pin "2")
@@
       (effects (font (size 1.27 1.27)) hide)
     )
+    (property "PN" "CC0402KRX7R7BB104" (at 196.85 29.21 0)
+      (effects (font (size 1.27 1.27)) hide)
+    )
     (pin "1")
     (pin "2")
@@
       (effects (font (size 1.27 1.27)) hide)
     )
+    (property "PN" "RC0402FR-075K1L" (at 58.42 81.28 0)
+      (effects (font (size 1.27 1.27)) hide)
+    )
     (pin "1")
     (pin "2")
@@
       (effects (font (size 1.27 1.27)) hide)
     )
+    (property "PN" "CC0402KRX7R7BB104" (at 166.37 29.21 0)
+      (effects (font (size 1.27 1.27)) hide)
+    )
     (pin "1")
     (pin "2")
@@
     )
     (property "Datasheet" "~" (at 120.65 57.15 0)
+      (effects (font (size 1.27 1.27)) hide)
+    )
+    (property "PN" "RC0402FR-071ML" (at 120.65 57.15 0)
       (effects (font (size 1.27 1.27)) hide)
     )
@@
       (effects (font (size 1.27 1.27)) hide)
     )
+    (property "PN" "CC0402KRX7R7BB104" (at 186.69 29.21 0)
+      (effects (font (size 1.27 1.27)) hide)
+    )
     (pin "1")
     (pin "2")
@@
       (effects (font (size 1.27 1.27)) hide)
     )
+    (property "PN" "RC0402FR-0722RL" (at 181.61 76.2 0)
+      (effects (font (size 1.27 1.27)) hide)
+    )
     (pin "1")
     (pin "2")
@@
       (effects (font (size 1.27 1.27)) hide)
     )
+    (property "PN" "CC0402KRX7R7BB104" (at 60.96 38.1 0)
+      (effects (font (size 1.27 1.27)) hide)
+    )
     (pin "1")
     (pin "2")
@@
     )
     (property "Datasheet" "~" (at 105.41 60.96 0)
+      (effects (font (size 1.27 1.27)) hide)
+    )
+    (property "PN" "CC0402JRNPO9BN220" (at 105.41 60.96 0)
       (effects (font (size 1.27 1.27)) hide)
     )
@@
       (effects (font (size 1.27 1.27)) hide)
     )
+    (property "PN" "CC0402KRX7R7BB104" (at 176.53 29.21 0)
+      (effects (font (size 1.27 1.27)) hide)
+    )
     (pin "1")
     (pin "2")
@@
       (effects (font (size 1.27 1.27)) hide)
     )
+    (property "PN" "RC0402FR-071K5L" (at 185.42 66.04 0)
+      (effects (font (size 1.27 1.27)) hide)
+    )
     (pin "1")
     (pin "2")
@@
       (effects (font (size 1.27 1.27)) hide)
     )
+    (property "PN" "RC0402FR-0710KL" (at 132.08 43.18 0)
+      (effects (font (size 1.27 1.27)) hide)
+    )
     (pin "1")
     (pin "2")
@@
     )
     (property "Datasheet" "~" (at 52.07 134.62 0)
+      (effects (font (size 1.27 1.27)) hide)
+    )
+    (property "PN" "DNP" (at 52.07 134.62 0)
       (effects (font (size 1.27 1.27)) hide)
     )
@@
       (effects (font (size 1.27 1.27)) hide)
     )
+    (property "PN" "RC0402FR-0710KL" (at 232.41 63.5 0)
+      (effects (font (size 1.27 1.27)) hide)
+    )
     (pin "1")
     (pin "2")
@@
       (effects (font (size 1.27 1.27)) hide)
     )
+    (property "PN" "CC0402ZRY5V6BB105" (at 91.44 38.1 0)
+      (effects (font (size 1.27 1.27)) hide)
+    )
     (pin "1")
     (pin "2")
@@
       (effects (font (size 1.27 1.27)) hide)
     )
+    (property "PN" "RC0402FR-0722RL" (at 181.61 73.66 0)
+      (effects (font (size 1.27 1.27)) hide)
+    )
     (pin "1")
     (pin "2")
@@
       (effects (font (size 1.27 1.27)) hide)
     )
+    (property "PN" "CC0402KRX5R6BB475" (at 55.88 38.1 0)
+      (effects (font (size 1.27 1.27)) hide)
+    )
     (pin "1")
     (pin "2")
@@
     )
     (property "Datasheet" "~" (at 105.41 53.34 0)
+      (effects (font (size 1.27 1.27)) hide)
+    )
+    (property "PN" "CC0402JRNPO9BN220" (at 105.41 53.34 0)
       (effects (font (size 1.27 1.27)) hide)
     )
@@
       (effects (font (size 1.27 1.27)) hide)
     )
+    (property "PN" "RC0402FR-0710KL" (at 232.41 85.09 0)
+      (effects (font (size 1.27 1.27)) hide)
+    )
